File: try3.kicad_pcb (KiCad board)
At the start: 2 copper layers, 442.9 x 144.5 mm, 224 parts, among them J1 USB_C_Receptacle, SW1 SW_Push, U1 AT90USB1286-AU, X1 XTAL_GND

Commit message: updated schematic and pcb
Parts:
- removed C5: 4.7u, Capacitor_SMD:C_0805_2012Metric_Pad1.18x1.45mm_HandSolder
- added LED1: LED, LED_SMD:LED_0805_2012Metric_Pad1.15x1.40mm_HandSolder, F.Cu at (447.4, -114.2)
- added LED2: LED, LED_SMD:LED_0805_2012Metric_Pad1.15x1.40mm_HandSolder, F.Cu at (447.4, -116.2)
- added LED3: LED, LED_SMD:LED_0805_2012Metric_Pad1.15x1.40mm_HandSolder, F.Cu at (447.4, -118.2)
- added R5: 22, Resistor_SMD:R_0805_2012Metric_Pad1.20x1.40mm_HandSolder, F.Cu at (390.2, -135.5)
- added R6: 22, Resistor_SMD:R_0805_2012Metric_Pad1.20x1.40mm_HandSolder, F.Cu at (390.2, -137.5)
- added R7: 260, Resistor_SMD:R_0805_2012Metric_Pad1.20x1.40mm_HandSolder, F.Cu at (453.6, -114.2)
- added R8: 260, Resistor_SMD:R_0805_2012Metric_Pad1.20x1.40mm_HandSolder, F.Cu at (453.6, -116.2)
- added R9: 260, Resistor_SMD:R_0805_2012Metric_Pad1.20x1.40mm_HandSolder, F.Cu at (453.6, -118.2)
- C4: value 0.1u -> 1u
- U1: footprint Package_QFP:TQFP-64_14x14mm_P0.8mm -> AT90USB1286AU:AT90USB1286-AU
- X1: value XTAL_GND -> Crystal_GND24
- moved C1 45.4 mm to (428.4, -100.5), turned to 270 degrees
- moved C3 43.0 mm to (435.7, -107.8), turned to 0 degrees
- moved C2 38.4 mm to (433.6, -121.7), turned to 0 degrees
- moved R2 20.7 mm to (378.2, -129.0), turned to 90 degrees
- moved C4 20.0 mm to (381.2, -129.0), turned to 270 degrees
- moved R1 14.0 mm to (384.4, -129.0), turned to 90 degrees
- moved C6 2.82 mm to (417.5, -128.7), turned to 180 degrees
- moved SW1 2.53 mm to (449.8, -125.4)
- moved C7 2.27 mm to (429.1, -127.9), turned to 0 degrees
- moved R3 2.20 mm to (438.8, -121.6), turned to 0 degrees
- moved X1 2.00 mm to (423.3, -128.2), turned to 315 degrees
- moved C8 0.51 mm to (435.7, -111.0), turned to 0 degrees
Connections:
- net Net-(C6-Pad1) renamed /XTAL-
- C1 pad 2: +5V -> GND
- C2 pad 2: +5V -> GND
- C3 pad 2: +5V -> GND
- C4 pad 2: +5V -> GND
- C6 pad 2: +5V -> GND
- C7 pad 1: Net-(C7-Pad1) -> /XTAL+
- C7 pad 2: +5V -> GND
- C8 pad 2: +5V -> GND
- J1 pad A1: +5V -> GND
- J1 pad A12: +5V -> GND
- J1 pad A6: Net-(J1-PadA6) -> /USB_D1+
- J1 pad A7: Net-(J1-PadA7) -> /USB_D1-
- J1 pad A8: (no net) -> Net-(J1-PadA8)
- J1 pad B1: +5V -> GND
- J1 pad B12: +5V -> GND
- J1 pad B6: Net-(J1-PadA6) -> /USB_D1+
- J1 pad B7: Net-(J1-PadA7) -> /USB_D1-
- J1 pad B8: (no net) -> Net-(J1-PadB8)
- J1 pad S1: +5V -> GND
- R1 pad 1: +5V -> GND
- R2 pad 1: +5V -> GND
- R4 pad 1: +5V -> GND
- SW1 pad 1: +5V -> GND
- U1 pad 10: (no net) -> /row5
- U1 pad 11: (no net) -> /LED1
- U1 pad 12: (no net) -> /LED2
- U1 pad 13: (no net) -> /LED3
- U1 pad 14: (no net) -> Net-(U1-Pad14)
- U1 pad 15: (no net) -> Net-(U1-Pad15)
- U1 pad 16: (no net) -> Net-(U1-Pad16)
- U1 pad 17: (no net) -> Net-(U1-Pad17)
- U1 pad 18: (no net) -> Net-(U1-Pad18)
- U1 pad 19: (no net) -> Net-(U1-Pad19)
- U1 pad 22: +5V -> GND
- U1 pad 23: Net-(C7-Pad1) -> /XTAL+
- U1 pad 25: (no net) -> Net-(U1-Pad25)
- U1 pad 26: (no net) -> Net-(U1-Pad26)
- U1 pad 27: (no net) -> Net-(U1-Pad27)
- U1 pad 28: (no net) -> Net-(U1-Pad28)
- U1 pad 29: (no net) -> Net-(U1-Pad29)
- U1 pad 30: (no net) -> Net-(U1-Pad30)
- U1 pad 31: (no net) -> Net-(U1-Pad31)
- U1 pad 32: (no net) -> Net-(U1-Pad32)
- U1 pad 33: Net-(J1-PadA5) -> Net-(U1-Pad33)
- U1 pad 34: Net-(J1-PadB5) -> Net-(U1-Pad34)
- U1 pad 4: Net-(J1-PadA7) -> /USB_D-
- U1 pad 5: Net-(J1-PadA6) -> /USB_D+
- U1 pad 53: +5V -> GND
- U1 pad 6: +5V -> GND
- U1 pad 62: (no net) -> Net-(U1-Pad62)
- U1 pad 63: +5V -> GND
- U1 pad 9: /row5 -> Net-(U1-Pad9)
- X1 pad 2: Net-(C7-Pad1) -> GND
- X1 pad 3: +5V -> /XTAL+
- X1 pad 4: (no net) -> GND
Routing:
- net VCC: track 127.0 -> 32.1 mm
- net Net-(J1-PadA7): track 92.3 -> 0.00 mm, vias 2 -> 0
- net Net-(J1-PadA6): track 88.5 -> 0.00 mm, vias 2 -> 0
- net /USB_D+: track 0.00 -> 55.0 mm, vias 0 -> 2
- net /USB_D-: track 0.00 -> 54.8 mm, vias 0 -> 2
- net +5V: track 52.0 -> 0.00 mm, vias 3 -> 0
- net Net-(J1-PadB5): track 53.2 -> 11.1 mm
- net Net-(J1-PadA5): track 38.8 -> 4.39 mm
- net GND: track 0.00 -> 18.6 mm
- net /LED3: track 0.00 -> 17.3 mm
- net /LED2: track 0.00 -> 16.9 mm
- net /LED1: track 0.00 -> 16.4 mm
- net /XTAL+: track 0.00 -> 12.4 mm
- net /USB_D1+: track 0.00 -> 11.1 mm
- net /USB_D1-: track 0.00 -> 10.1 mm
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- added copper zone on F.Cu, net GND
- added copper zone on B.Cu, net VCC
- removed copper zone on B.Cu, net +5V
- removed copper zone on F.Cu, net +5V
Other:
- outline, holes or cut-outs redrawn
