File: try3.sch (KiCad schematic (older format))
At the start: 224 parts, among them J1 USB_C_Receptacle, SW1 SW_Push, U1 AT90USB1286-AU, X1 XTAL_GND

Commit message: updated schematic and pcb
Parts:
- removed C5: 4.7u, Capacitor_SMD:C_0805_2012Metric_Pad1.18x1.45mm_HandSolder, symbol Device:C
- removed X1: XTAL_GND, Crystal:Crystal_SMD_SeikoEpson_TSX3225-4Pin_3.2x2.5mm_HandSoldering, symbol keyboard_parts:XTAL_GND
- added LED1, LED2, LED3: LED, LED_SMD:LED_0805_2012Metric_Pad1.15x1.40mm_HandSolder, symbol Device:LED
- added R5, R6: 22, Resistor_SMD:R_0805_2012Metric_Pad1.20x1.40mm_HandSolder, symbol Device:R
- added R7, R8, R9: 260, Resistor_SMD:R_0805_2012Metric_Pad1.20x1.40mm_HandSolder, symbol Device:R
- added X1: Crystal_GND24, Crystal:Crystal_SMD_SeikoEpson_TSX3225-4Pin_3.2x2.5mm_HandSoldering, symbol Device:Crystal_GND24
- C4: value 0.1u -> 1u
- U1: footprint Package_QFP:TQFP-64_14x14mm_P0.8mm -> AT90USB1286AU:AT90USB1286-AU
Connections:
- net row5: now also U1.10 (PB0); no longer U1.9 (PE3)
- net LED1: now reaches U1.11 (PB1)
- net LED1: now also LED1.2 (A)
- net LED2: now reaches U1.12 (PB2)
- net LED2: now also LED2.2 (A)
- net LED3: now reaches U1.13 (PB3)
- net LED3: now also LED3.2 (A)
- net XTAL+: now reaches C7.1, U1.23 (XTAL2)
- net XTAL+: now also X1.3
- net XTAL-: now reaches C6.1, U1.24 (XTAL1)
- net XTAL-: now also X1.1
- net at J1.A5 (CC1), R1.2: no longer U1.33 (PE0)
- net at J1.B5 (CC2), R2.2: no longer U1.34 (PE1)
- net USB_D1-: now reaches J1.A7 (D-), J1.B7 (D-)
- net USB_D1-: now also R5.2; no longer U1.4 (D-)
- net USB_D1+: now reaches J1.A6 (D+), J1.B6 (D+)
- net USB_D1+: now also R6.2; no longer U1.5 (D+)
- net +5V renamed GND
- net GND: now also R7.2, R8.2, R9.2, X1.2, X1.4
- new net: LED1.1 (K), R7.1
- new net: LED2.1 (K), R8.1
- new net: LED3.1 (K), R9.1
- new net USB_D+: R6.1, U1.5 (D+)
- new net USB_D-: R5.1, U1.4 (D-)
- no-connect marks 29 -> 25
Other:
- moved on the sheet: C1, C2, C3, C6, C7, R1, R2, R3, R4, SW1
