File: 100-mk-pcb.kicad_pcb (KiCad board)
At the start: 2 copper layers, 442.9 x 144.5 mm, 231 parts, among them J1 USB_C_Receptacle, SW1 SW_Push, U1 AT90USB1286-AU, X1 Crystal_GND24

Commit message: backup edited files
Parts:
- CAPS LOCK: renamed from LED3
- D1, D10, D100, D101, D102, D103, D104, D11, D12, D13, D14, D15, D16, D17, D18, D19, D2, D20, D21, D22, D23, D24, D25, D26, D27, D28, D29, D3, D30, D31, D32, D33, D34, D35, D36, D37, D38, D39, D4, D40, D41, D42, D43, D44, D45, D46, D47, D48, D49, D5, D50, D51, D52, D53, D54, D55, D56, D57, D58, D59, D6, D60, D61, D62, D63, D64, D65, D66, D67, D68, D69, D7, D70, D71, D72, D73, D74, D75, D76, D77, D78, D79, D8, D80, D81, D82, D83, D84, D85, D86, D87, D88, D89, D9, D90, D91, D92, D93, D94, D95, D96, D97, D98, D99: moved to F.Cu
- K_1, K_10, K_100, K_101, K_102, K_11, K_13, K_14, K_15, K_16, K_17, K_19, K_2, K_20, K_21, K_22, K_23, K_24, K_25, K_26, K_27, K_28, K_29, K_30, K_31, K_32, K_33, K_35, K_36, K_37, K_38, K_39, K_40, K_41, K_42, K_43, K_44, K_45, K_46, K_47, K_48, K_49, K_50, K_51, K_52, K_53, K_55, K_56, K_57, K_58, K_59, K_61, K_62, K_63, K_64, K_66, K_67, K_68, K_69, K_7, K_75, K_76, K_77, K_78, K_79, K_8, K_80, K_81, K_82, K_83, K_84, K_85, K_86, K_87, K_88, K_89, K_9, K_90, K_91, K_93, K_94, K_95, K_96, K_97, K_98, K_99: footprint Button_Switch_Keyboard:SW_Cherry_MX_1.00u_PCB -> Button_Switch_Keyboard:SW_Cherry_MX_1.00u_Plate
- K_103, K_104: footprint Button_Switch_Keyboard:SW_Cherry_MX_2.00u_Vertical_PCB -> Button_Switch_Keyboard:SW_Cherry_MX_2.00u_Vertical_Plate
- K_12, K_60, K_65: footprint Button_Switch_Keyboard:SW_Cherry_MX_1.00u_PCB -> Button_Switch_Keyboard:SW_Cherry_MX_1.25u_Plate
- K_18: footprint Button_Switch_Keyboard:SW_Cherry_MX_1.25u_PCB -> Button_Switch_Keyboard:SW_Cherry_MX_1.25u_Plate
- K_3, K_71: footprint Button_Switch_Keyboard:SW_Cherry_MX_1.50u_PCB -> Button_Switch_Keyboard:SW_Cherry_MX_1.50u_Plate
- K_34: footprint Button_Switch_Keyboard:SW_Cherry_MX_6.25u_PCB -> Button_Switch_Keyboard:SW_Cherry_MX_6.25u_Plate
- K_4: footprint Button_Switch_Keyboard:SW_Cherry_MX_1.75u_PCB -> Button_Switch_Keyboard:SW_Cherry_MX_1.75u_Plate
- K_5, K_72: footprint Button_Switch_Keyboard:SW_Cherry_MX_2.25u_PCB -> Button_Switch_Keyboard:SW_Cherry_MX_2.25u_Plate
- K_54, K_6, K_74: footprint Button_Switch_Keyboard:SW_Cherry_MX_1.50u_PCB -> Button_Switch_Keyboard:SW_Cherry_MX_1.25u_Plate
- K_70, K_92: footprint Button_Switch_Keyboard:SW_Cherry_MX_2.00u_PCB -> Button_Switch_Keyboard:SW_Cherry_MX_2.00u_Plate
- K_73: footprint Button_Switch_Keyboard:SW_Cherry_MX_2.75u_PCB -> Button_Switch_Keyboard:SW_Cherry_MX_2.75u_Plate
- NUM LOCK: renamed from LED1
- SCROLL LOCK: renamed from LED2
- SW1: value SW_Push -> SW_Reset
- moved D12 12.9 mm to (49.0, -10.0), turned to 90 degrees
- moved D6 12.7 mm to (25.5, -10.0), turned to 90 degrees
- moved D60 12.4 mm to (239.0, -10.0), turned to 90 degrees
- moved D54 12.2 mm to (215.5, -10.0), turned to 90 degrees
- moved D5 10.4 mm to (35.0, -29.0), turned to 90 degrees
- moved D78 10.4 mm to (314.5, -10.0), turned to 90 degrees
- moved D34 10.4 mm to (144.0, -10.0), turned to 90 degrees
- moved D83 10.4 mm to (333.5, -10.0), turned to 90 degrees
- moved D95 10.3 mm to (397.5, -48.0), turned to 90 degrees
- moved D35 10.3 mm to (163.0, -119.0), turned to 90 degrees
- moved D92 10.3 mm to (388.0, -10.0), turned to 90 degrees
- moved D96 10.3 mm to (397.5, -29.0), turned to 90 degrees
- moved D18 10.3 mm to (73.0, -10.0), turned to 90 degrees
- moved D53 10.3 mm to (217.5, -29.0), turned to 90 degrees
- moved D32 10.3 mm to (132.2, -48.0), turned to 90 degrees
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Routing:
- net /row5: track 543.4 -> 549.0 mm
- net /row2: track 509.3 -> 505.7 mm, vias 0 -> 1
- net /row1: track 477.9 -> 475.4 mm, vias 0 -> 1
- net /col1: track 488.6 -> 491.0 mm
- net /row3: track 501.6 -> 503.6 mm
- net /row4: track 532.2 -> 530.3 mm
- net Net-(D52-Pad2): track 6.97 -> 5.69 mm
- net Net-(D28-Pad2): track 6.97 -> 5.69 mm
- net Net-(D84-Pad2): track 6.97 -> 5.70 mm
- net Net-(D27-Pad2): track 6.97 -> 5.70 mm
- net Net-(D8-Pad2): track 6.97 -> 5.70 mm
- net Net-(D1-Pad2): track 6.97 -> 5.72 mm
- net Net-(D24-Pad2): track 6.97 -> 5.72 mm
- net Net-(D90-Pad2): track 6.97 -> 5.73 mm
- net Net-(D85-Pad2): track 6.97 -> 5.73 mm
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Other:
- net class Default removed
- board text added: "SW_Reset"
